Commit message: UPDATE: shows something

File: first_model/urdf/first_model.urdf.xacro (robot description, xacro)
@@ -3,5 +3,5 @@
     <xacro:property name="wheel_r" value="0.20"/>
     <xacro:property name="wheel_width" value="0.05"/>
-    <xacro:property name="pi" value="3.1415" />
+<!--    <xacro:property name="pi" value="3.1415" />-->
     <material name="black">
         <color rgba="0 0 0 1"/>
@@ -18,5 +18,5 @@
                 <origin xyz="0 0 0" rpy="${pi/2} 0 0"/>
                 <geometry>
-                    <cylinder radius="${wheel_r}" length="{wheel_width}"/>
+                    <cylinder radius="${wheel_r}" length="${wheel_width}"/>
                 </geometry>
                 <material name="black"/>
@@ -25,8 +25,8 @@
                 <origin xyz="0 0 0" rpy="${pi/2} 0 0"/>
                 <geometry>
-                    <cylinder radius="${wheel_r}" length="{wheel_width}"/>
+                    <cylinder radius="${wheel_r}" length="${wheel_width}"/>
                 </geometry>
             </collision>
-            <xacro:default_inertia mass="1"/>
+            <xacro:default_inertial mass="1"/>
         </link>
         <joint name="${prefix}_${sufix}_wheel_joint" type="continuous">
@@ -41,5 +41,5 @@
             <origin xyz="0 0 ${wheel_r+0.5}" rpy="${pi/2} 0 0"/>
             <geometry>
-                <cylinder radius="${wheel_r}" length="{wheel_width}"/>
+                <cylinder radius="${wheel_r}" length="${wheel_width}"/>
             </geometry>
             <material name="black"/>
@@ -47,8 +47,8 @@
         <collision>
             <geometry>
-                <cylinder radius="${wheel_r}" length="{wheel_width}"/>
+                <cylinder radius="${wheel_r}" length="${wheel_width}"/>
             </geometry>
         </collision>
-        <xacro:default_inertia mass="1"/>
+        <xacro:default_inertial mass="1"/>
     </link>
 </robot>

Commit message: UPDATE: good position

File: first_model/urdf/first_model.urdf.xacro (robot description, xacro)
@@ -39,5 +39,5 @@
     <link name="wheel">
         <visual>
-            <origin xyz="0 0 ${wheel_r+0.5}" rpy="${pi/2} 0 0"/>
+            <origin xyz="0 0 ${wheel_r}" rpy="${pi/2} 0 0"/>
             <geometry>
                 <cylinder radius="${wheel_r}" length="${wheel_width}"/>

Commit message: UPDATE: cleaned a bit and made sure it actually works

File: first_model/urdf/first_model.urdf.xacro (robot description, xacro)
@@ -3,5 +3,5 @@
     <xacro:property name="wheel_r" value="0.20"/>
     <xacro:property name="wheel_width" value="0.05"/>
-<!--    <xacro:property name="pi" value="3.1415" />-->
+    <!--    <xacro:property name="pi" value="3.1415" />-->
     <material name="black">
         <color rgba="0 0 0 1"/>

Commit message: UPDATE: starting with a box

File: first_model/urdf/first_model.urdf.xacro (robot description, xacro)
@@ -3,5 +3,7 @@
     <xacro:property name="wheel_r" value="0.20"/>
     <xacro:property name="wheel_width" value="0.05"/>
-    <!--    <xacro:property name="pi" value="3.1415" />-->
+    <xacro:property name="base_length" value="1"/>
+    <xacro:property name="base_width" value="1"/>
+    <xacro:property name="base_height" value="1"/>
     <material name="black">
         <color rgba="0 0 0 1"/>
@@ -13,5 +15,5 @@
         </inertial>
     </xacro:macro>
-    <xacro:macro name="wheel" params="prefix sufix reflect:=1">
+    <xacro:macro name="wheel" params="prefix sufix reflect">
         <link name="${prefix}_${sufix}_wheel">
             <visual>
@@ -37,18 +39,19 @@
         </joint>
     </xacro:macro>
-    <link name="wheel">
+    <link name="base">
         <visual>
-            <origin xyz="0 0 ${wheel_r}" rpy="${pi/2} 0 0"/>
+            <origin xyz="0 0 ${base_height}/2"/>
             <geometry>
-                <cylinder radius="${wheel_r}" length="${wheel_width}"/>
+                <box size="${base_length} ${base_width}  ${base_height}"/>
             </geometry>
             <material name="black"/>
         </visual>
         <collision>
+            <origin xyz="0 0 ${base_height}/2"/>
             <geometry>
-                <cylinder radius="${wheel_r}" length="${wheel_width}"/>
+                <box size="${base_length} ${base_width}  ${base_height}"/>
             </geometry>
         </collision>
-        <xacro:default_inertial mass="1"/>
+        <xacro:default_inertial mass="10"/>
     </link>
 </robot>

File: first_model/urdf/robot.urdf (robot description, URDF)
Before this commit: robot hybrid_robot, 1 links, 0 joints
Links:
- removed link wheel
- added link base; collision box size=1 1 1; visual box size=0 0 0

Commit message: UPDATE: set correct inertia with current box

File: first_model/urdf/first_model.urdf.xacro (robot description, xacro)
@@ -1,9 +1,9 @@
 <?xml version="1.0"?>
 <robot name="hybrid_robot" xmlns:xacro="http://ros.org/wiki/xacro">
-    <xacro:property name="wheel_r" value="0.20"/>
-    <xacro:property name="wheel_width" value="0.05"/>
+    <xacro:property name="wheel_r" value="0.10"/>
+    <xacro:property name="wheel_width" value="0.02"/>
     <xacro:property name="base_length" value="1"/>
-    <xacro:property name="base_width" value="1"/>
-    <xacro:property name="base_height" value="1"/>
+    <xacro:property name="base_width" value="0.5"/>
+    <xacro:property name="base_height" value="0.1"/>
     <material name="black">
         <color rgba="0 0 0 1"/>
@@ -41,5 +41,5 @@
     <link name="base">
         <visual>
-            <origin xyz="0 0 ${base_height}/2"/>
+            <origin xyz="0 0 ${wheel_r}"/>
             <geometry>
                 <box size="${base_length} ${base_width}  ${base_height}"/>
@@ -48,10 +48,13 @@
         </visual>
         <collision>
-            <origin xyz="0 0 ${base_height}/2"/>
+            <origin xyz="0 0 ${wheel_r}"/>
             <geometry>
                 <box size="${base_length} ${base_width}  ${base_height}"/>
             </geometry>
         </collision>
-        <xacro:default_inertial mass="10"/>
+        <inertial>
+            <mass value="10"/>
+            <inertia ixx="0.21666666666666667" ixy="0" ixz="0" iyy="0.8416666666666667" iyz="0" izz="1.0416666666666665"/>
+        </inertial>
     </link>
 </robot>

Commit message: UPDATE: a box with 4 wheels

File: first_model/urdf/first_model.urdf.xacro (robot description, xacro)
@@ -15,8 +15,7 @@
         </inertial>
     </xacro:macro>
-    <xacro:macro name="wheel" params="prefix sufix reflect">
-        <link name="${prefix}_${sufix}_wheel">
+    <xacro:macro name="wheel" params="position side parent">
+        <link name="${position}_${side}_wheel">
             <visual>
-                <origin xyz="0 0 0" rpy="${pi/2} 0 0"/>
                 <geometry>
                     <cylinder radius="${wheel_r}" length="${wheel_width}"/>
@@ -25,5 +24,4 @@
             </visual>
             <collision>
-                <origin xyz="0 0 0" rpy="${pi/2} 0 0"/>
                 <geometry>
                     <cylinder radius="${wheel_r}" length="${wheel_width}"/>
@@ -32,14 +30,21 @@
             <xacro:default_inertial mass="1"/>
         </link>
-        <joint name="${prefix}_${sufix}_wheel_joint" type="continuous">
+        <joint name="${position}_${side}_wheel_joint" type="continuous">
+            <xacro:property name="origin_x" value="${base_length*(1/2-1/4)}"/>
+            <xacro:if value="${position == 'back'}">
+                <xacro:property name="origin_x" value="${-base_length*(1/2-1/4)}"/>
+            </xacro:if>
+            <xacro:property name="origin_y" value="${(base_width + wheel_width)/2}"/>
+            <xacro:if value="${side == 'right'}">
+                <xacro:property name="origin_y" value="${-(base_width + wheel_width)/2}"/>
+            </xacro:if>
             <axis xyz="0 1 0" rpy="0 0 0"/>
-            <parent link="${prefix}_base"/>
-            <child link="${prefix}_${sufix}_wheel"/>
-            <origin xyz="0 0 -${wheel_r+wheel_width/2}" rpy="0 0 0"/>
+            <parent link="${parent}"/>
+            <child link="${position}_${side}_wheel"/>
+            <origin xyz="${origin_x} ${origin_y} 0" rpy="${pi/2} 0 0"/>
         </joint>
     </xacro:macro>
     <link name="base">
         <visual>
-            <origin xyz="0 0 ${wheel_r}"/>
             <geometry>
                 <box size="${base_length} ${base_width}  ${base_height}"/>
@@ -58,3 +63,7 @@
         </inertial>
     </link>
+    <xacro:wheel position="front" side="right" parent="base"/>
+    <xacro:wheel position="front" side="left" parent="base"/>
+    <xacro:wheel position="back" side="right" parent="base"/>
+    <xacro:wheel position="back" side="left" parent="base"/>
 </robot>

Commit message: UPDATE: 2 bodies with 4 wheels

File: first_model/urdf/first_model.urdf.xacro (robot description, xacro)
@@ -1,9 +1,12 @@
 <?xml version="1.0"?>
 <robot name="hybrid_robot" xmlns:xacro="http://ros.org/wiki/xacro">
-    <xacro:property name="wheel_r" value="0.10"/>
+    <xacro:property name="wheel_r" value="0.15"/>
     <xacro:property name="wheel_width" value="0.02"/>
     <xacro:property name="base_length" value="1"/>
     <xacro:property name="base_width" value="0.5"/>
     <xacro:property name="base_height" value="0.1"/>
+    <xacro:property name="extension_length" value="1"/>
+    <xacro:property name="extension_width" value="0.45"/>
+    <xacro:property name="extension_height" value="0.095"/>
     <material name="black">
         <color rgba="0 0 0 1"/>
@@ -31,11 +34,13 @@
         </link>
         <joint name="${position}_${side}_wheel_joint" type="continuous">
-            <xacro:property name="origin_x" value="${base_length*(1/2-1/4)}"/>
+            <xacro:property name="origin_x" value="${base_length/2-0.05}"/>
             <xacro:if value="${position == 'back'}">
-                <xacro:property name="origin_x" value="${-base_length*(1/2-1/4)}"/>
+                <xacro:property name="origin_x" value="${-(base_length/2-0.05)}"/>
             </xacro:if>
             <xacro:property name="origin_y" value="${(base_width + wheel_width)/2}"/>
             <xacro:if value="${side == 'right'}">
                 <xacro:property name="origin_y" value="${-(base_width + wheel_width)/2}"/>
+            </xacro:if>
+            <xacro:if value="${parent == 'extension'}">
             </xacro:if>
             <axis xyz="0 1 0" rpy="0 0 0"/>
@@ -53,5 +58,4 @@
         </visual>
         <collision>
-            <origin xyz="0 0 ${wheel_r}"/>
             <geometry>
                 <box size="${base_length} ${base_width}  ${base_height}"/>
@@ -63,7 +67,31 @@
         </inertial>
     </link>
+    <link name="extension">
+        <visual>
+            <geometry>
+                <box size="${extension_length} ${extension_width} ${extension_height}"/>
+            </geometry>
+            <material name="balck"/>
+        </visual>
+        <collision>
+            <geometry>
+                <box size="${extension_length} ${extension_width} ${extension_height}"/>
+            </geometry>
+        </collision>
+        <inertial>
+            <mass value="10"/>
+            <inertia ixx="0.9208333333333332" ixy="0" ixz="0" iyy="1.5854166666666663" iyz="0" izz="1.0020833333333334"/>
+        </inertial>
+    </link>
+    <joint name="extension_base_joint" type="prismatic">
+        <axis xyz="1 0 0"/>
+        <parent link="base"/>
+        <child link="extension"/>
+        <origin xyz="-.1 0 0"/>
+        <limit lower="0" upper="1" effort="100" velocity="10"/>
+    </joint>
     <xacro:wheel position="front" side="right" parent="base"/>
     <xacro:wheel position="front" side="left" parent="base"/>
-    <xacro:wheel position="back" side="right" parent="base"/>
-    <xacro:wheel position="back" side="left" parent="base"/>
+    <xacro:wheel position="back" side="right" parent="extension"/>
+    <xacro:wheel position="back" side="left" parent="extension"/>
 </robot>

Commit message: UPDATE: fix inertial tensor for the extension

File: first_model/urdf/first_model.urdf.xacro (robot description, xacro)
@@ -72,5 +72,5 @@
                 <box size="${extension_length} ${extension_width} ${extension_height}"/>
             </geometry>
-            <material name="balck"/>
+            <material name="black"/>
         </visual>
         <collision>
@@ -81,5 +81,5 @@
         <inertial>
             <mass value="10"/>
-            <inertia ixx="0.9208333333333332" ixy="0" ixz="0" iyy="1.5854166666666663" iyz="0" izz="1.0020833333333334"/>
+            <inertia ixx="0.17627083333333335" ixy="0" ixz="0" iyy="0.8408541666666667" iyz="0" izz="1.0020833333333334"/>
         </inertial>
     </link>

File: first_model/urdf/robot.urdf (robot description, URDF)
Before this commit: robot hybrid_robot, 1 links, 0 joints
Links:
- added link back_left_wheel, mass 1; collision cylinder length=0.02 radius=0.15; visual cylinder length=0.02 radius=0.15
- added link back_right_wheel, mass 1; collision cylinder length=0.02 radius=0.15; visual cylinder length=0.02 radius=0.15
- added link extension, mass 10; collision box size=1 0.45 0.095; visual box size=1 0.45 0.095
- added link front_left_wheel, mass 1; collision cylinder length=0.02 radius=0.15; visual cylinder length=0.02 radius=0.15
- added link front_right_wheel, mass 1; collision cylinder length=0.02 radius=0.15; visual cylinder length=0.02 radius=0.15
- link base: mass None -> 10; geometry collision box size=1 0.5 0.1; visual box size=1 0.5 0.1
Joints:
- added joint back_left_wheel_joint: type continuous, parent extension, child back_left_wheel, origin xyz=-0.45 0.26 0 rpy=1.5707963267948966 0 0, axis 0 1 0
- added joint back_right_wheel_joint: type continuous, parent extension, child back_right_wheel, origin xyz=-0.45 -0.26 0 rpy=1.5707963267948966 0 0, axis 0 1 0
- added joint extension_base_joint: type prismatic, parent base, child extension, origin xyz=-.1 0 0, axis 1 0 0, limit lower=0 upper=1 effort=100 velocity=10
- added joint front_left_wheel_joint: type continuous, parent base, child front_left_wheel, origin xyz=0.45 0.26 0 rpy=1.5707963267948966 0 0, axis 0 1 0
- added joint front_right_wheel_joint: type continuous, parent base, child front_right_wheel, origin xyz=0.45 -0.26 0 rpy=1.5707963267948966 0 0, axis 0 1 0

Commit message: UPDATE: correct wheels inertia and added the transmission to the xacro

File: first_model/urdf/first_model.urdf.xacro (robot description, xacro)
@@ -12,10 +12,10 @@
         <color rgba="0 0 0 1"/>
     </material>
-    <xacro:macro name="default_inertial" params="mass">
-        <inertial>
-            <mass value="${mass}"/>
-            <inertia ixx="1.0" ixy="0.0" ixz="0.0" iyy="1.0" iyz="0.0" izz="1.0"/>
-        </inertial>
-    </xacro:macro>
+    <material name="red">
+        <color rgba="1 0 0 1"/>
+    </material>
+    <material name="blue">
+        <color rgba="0 0 1 1"/>
+    </material>
     <xacro:macro name="wheel" params="position side parent">
         <link name="${position}_${side}_wheel">
@@ -31,5 +31,8 @@
                 </geometry>
             </collision>
-            <xacro:default_inertial mass="1"/>
+            <inertial>
+                <mass value="1"/>
+                <inertia ixx="0.005658333333333333" ixy="0" ixz="0" iyy="0.005658333333333333" iyz="0" izz="0.01125"/>
+            </inertial>
         </link>
         <joint name="${position}_${side}_wheel_joint" type="continuous">
@@ -55,5 +58,5 @@
                 <box size="${base_length} ${base_width}  ${base_height}"/>
             </geometry>
-            <material name="black"/>
+            <material name="blue"/>
         </visual>
         <collision>
@@ -72,5 +75,5 @@
                 <box size="${extension_length} ${extension_width} ${extension_height}"/>
             </geometry>
-            <material name="black"/>
+            <material name="red"/>
         </visual>
         <collision>
@@ -88,6 +91,6 @@
         <parent link="base"/>
         <child link="extension"/>
-        <origin xyz="-.1 0 0"/>
-        <limit lower="0" upper="1" effort="100" velocity="10"/>
+        <origin xyz="-0.1 0 0"/>
+        <limit lower="-0.9" upper="0" effort="100" velocity="10"/>
     </joint>
     <xacro:wheel position="front" side="right" parent="base"/>
@@ -95,3 +98,58 @@
     <xacro:wheel position="back" side="right" parent="extension"/>
     <xacro:wheel position="back" side="left" parent="extension"/>
+    <transmission name="trans_extension_base_joint">
+        <type>transmission_interface/SimpleTransmission</type>
+        <joint name="extension_base_joint">
+            <hardwareInterface>hardware_interface/EffortJointInterface</hardwareInterface>
+        </joint>
+        <actuator name="extension_base_joint_motor">
+            <hardwareInterface>hardware_interface/EffortJointInterface</hardwareInterface>
+            <mechanicalReduction>1</mechanicalReduction>
+        </actuator>
+    </transmission>
+    <transmission name="trans_front_right_wheel_joint">
+        <type>transmission_interface/SimpleTransmission</type>
+        <joint name="front_right_wheel_joint">
+            <hardwareInterface>hardware_interface/EffortJointInterface</hardwareInterface>
+        </joint>
+        <actuator name="front_right_wheel_joint_motor">
+            <hardwareInterface>hardware_interface/EffortJointInterface</hardwareInterface>
+            <mechanicalReduction>1</mechanicalReduction>
+        </actuator>
+    </transmission>
+    <transmission name="trans_front_left_wheel_joint">
+        <type>transmission_interface/SimpleTransmission</type>
+        <joint name="front_left_wheel_joint">
+            <hardwareInterface>hardware_interface/EffortJointInterface</hardwareInterface>
+        </joint>
+        <actuator name="front_left_wheel_joint_motor">
+            <hardwareInterface>hardware_interface/EffortJointInterface</hardwareInterface>
+            <mechanicalReduction>1</mechanicalReduction>
+        </actuator>
+    </transmission>
+    <transmission name="trans_back_right_wheel_joint">
+        <type>transmission_interface/SimpleTransmission</type>
+        <joint name="back_right_wheel_joint">
+            <hardwareInterface>hardware_interface/EffortJointInterface</hardwareInterface>
+        </joint>
+        <actuator name="back_right_wheel_joint_motor">
+            <hardwareInterface>hardware_interface/EffortJointInterface</hardwareInterface>
+            <mechanicalReduction>1</mechanicalReduction>
+        </actuator>
+    </transmission>
+    <transmission name="trans_back_left_wheel_joint">
+        <type>transmission_interface/SimpleTransmission</type>
+        <joint name="back_left_wheel_joint">
+            <hardwareInterface>hardware_interface/EffortJointInterface</hardwareInterface>
+        </joint>
+        <actuator name="back_left_wheel_joint_motor">
+            <hardwareInterface>hardware_interface/EffortJointInterface</hardwareInterface>
+            <mechanicalReduction>1</mechanicalReduction>
+        </actuator>
+    </transmission>
+    <gazebo>
+        <plugin name="gazebo_ros_control" filename="libgazebo_ros_control.so">
+            <robotNamespace>/</robotNamespace>
+        </plugin>
+    </gazebo>
 </robot>
