Commit message: UPDATE: looks like it loads the controllers

File: hybrid_robot/first_model/urdf/robot.urdf (robot description, URDF)
Before this commit: robot hybrid_robot, 6 links, 5 joints
Joints:
- joint extension_base_joint: limit lower=0 upper=1 effort=100 velocity=10 -> lower=-0.9 upper=0 effort=100 velocity=10; origin xyz=-.1 0 0 -> xyz=-0.1 0 0
