Commit message: Working joint state controllers
Added new file control.launch to start the controllers
Added  a yaml file to hold configurations of joints hybrid_robotV0_2.yaml
small changes to diverse files, need to make the controllers to work

File: hybrid_jumping_robot/urdf/plugins.gazebo.xacro (robot description, xacro)
@@ -21,5 +21,5 @@
   <gazebo>
       <plugin filename="libgazebo_ros_control.so" name="gazebo_ros_control">
-          <robotNamespace>/hybrid_robotv0_2</robotNamespace>
+          <robotNamespace>/hybrid_robotV0_2</robotNamespace>
       </plugin>
   </gazebo>
@@ -27,5 +27,5 @@
     <plugin name="skid_steer_drive_controller" filename="libgazebo_ros_skid_steer_drive.so">
       <updateRate>100.0</updateRate>
-      <robotNamespace>/hybrid_robotv0_2</robotNamespace>
+      <robotNamespace>/hybrid_robotV0_2</robotNamespace>
       <leftFrontJoint>front_left_wheel_joint</leftFrontJoint>
       <rightFrontJoint>front_right_wheel_joint</rightFrontJoint>

File: hybrid_jumping_robot/urdf/transmission.xacro (robot description, xacro)
@@ -51,53 +51,3 @@
       </actuator>
   </transmission>
-  <transmission name="trans_extension_base_joint">
-      <type>transmission_interface/SimpleTransmission</type>
-      <joint name="extension_base_joint">
-          <hardwareInterface>hardware_interface/EffortJointInterface</hardwareInterface>
-      </joint>
-      <actuator name="extension_base_joint_motor">
-          <hardwareInterface>hardware_interface/EffortJointInterface</hardwareInterface>
-          <mechanicalReduction>1</mechanicalReduction>
-      </actuator>
-  </transmission>
-  <transmission name="trans_front_right_wheel_joint">
-      <type>transmission_interface/SimpleTransmission</type>
-      <joint name="front_right_wheel_joint">
-          <hardwareInterface>hardware_interface/EffortJointInterface</hardwareInterface>
-      </joint>
-      <actuator name="front_right_wheel_joint_motor">
-          <hardwareInterface>hardware_interface/EffortJointInterface</hardwareInterface>
-          <mechanicalReduction>1</mechanicalReduction>
-      </actuator>
-  </transmission>
-  <transmission name="trans_front_left_wheel_joint">
-      <type>transmission_interface/SimpleTransmission</type>
-      <joint name="front_left_wheel_joint">
-          <hardwareInterface>hardware_interface/EffortJointInterface</hardwareInterface>
-      </joint>
-      <actuator name="front_left_wheel_joint_motor">
-          <hardwareInterface>hardware_interface/EffortJointInterface</hardwareInterface>
-          <mechanicalReduction>1</mechanicalReduction>
-      </actuator>
-  </transmission>
-  <transmission name="trans_back_right_wheel_joint">
-      <type>transmission_interface/SimpleTransmission</type>
-      <joint name="back_right_wheel_joint">
-          <hardwareInterface>hardware_interface/EffortJointInterface</hardwareInterface>
-      </joint>
-      <actuator name="back_right_wheel_joint_motor">
-          <hardwareInterface>hardware_interface/EffortJointInterface</hardwareInterface>
-          <mechanicalReduction>1</mechanicalReduction>
-      </actuator>
-  </transmission>
-  <transmission name="trans_back_left_wheel_joint">
-      <type>transmission_interface/SimpleTransmission</type>
-      <joint name="back_left_wheel_joint">
-          <hardwareInterface>hardware_interface/EffortJointInterface</hardwareInterface>
-      </joint>
-      <actuator name="back_left_wheel_joint_motor">
-          <hardwareInterface>hardware_interface/EffortJointInterface</hardwareInterface>
-          <mechanicalReduction>1</mechanicalReduction>
-      </actuator>
-  </transmission>
 </robot>
