Commit message: Improved model
Made a more realistic model off what we can do

File: hybrid_jumping_robot/urdf/first_modelV0_2.urdf.xacro (robot description, xacro)
@@ -1,61 +1,95 @@
 <?xml version="1.0"?>
 <robot name="hybrid_robotv0_2" xmlns:xacro="http://ros.org/wiki/xacro">
-  <xacro:include filename="$(find hybrid_jumping_robot)/urdf/material.xacro"/>
-  <xacro:include filename="$(find hybrid_jumping_robot)/urdf/plugins.gazebo.xacro"/>
-  <xacro:include filename="$(find hybrid_jumping_robot)/urdf/macro.xacro"/>
-  <xacro:include filename="$(find hybrid_jumping_robot)/urdf/transmission.xacro"/>
-  <xacro:property name="wheel_r" value="0.15"/>
-  <xacro:property name="wheel_width" value="0.02"/>
-  <xacro:property name="base_length" value="1"/>
-  <xacro:property name="base_width" value="0.5"/>
-  <xacro:property name="base_height" value="0.1"/>
-  <xacro:property name="extension_length" value="1"/>
-  <xacro:property name="extension_width" value="0.45"/>
-  <xacro:property name="extension_height" value="0.095"/>
-  <link name="base">
-      <visual>
-          <geometry>
-              <box size="${base_length} ${base_width}  ${base_height}"/>
-          </geometry>
-          <material name="blue"/>
-      </visual>
-      <collision>
-          <geometry>
-              <box size="${base_length} ${base_width}  ${base_height}"/>
-          </geometry>
-      </collision>
-      <inertial>
-          <mass value="10"/>
-          <inertia ixx="0.21666666666666667" ixy="0" ixz="0" iyy="0.8416666666666667" iyz="0" izz="1.0416666666666665"/>
-      </inertial>
-  </link>
-  <link name="extension">
-      <visual>
-          <geometry>
-              <box size="${extension_length} ${extension_width} ${extension_height}"/>
-          </geometry>
-          <material name="red"/>
-      </visual>
-      <collision>
-          <geometry>
-              <box size="${extension_length} ${extension_width} ${extension_height}"/>
-          </geometry>
-      </collision>
-      <inertial>
-          <mass value="10"/>
-          <inertia ixx="0.17627083333333335" ixy="0" ixz="0" iyy="0.8408541666666667" iyz="0" izz="1.0020833333333334"/>
-      </inertial>
-  </link>
-  <joint name="extension_base_joint" type="prismatic">
-      <axis xyz="1 0 0"/>
-      <parent link="base"/>
-      <child link="extension"/>
-      <origin xyz="-0.1 0 0"/>
-      <limit lower="-0.9" upper="0" effort="10000" velocity="1000"/>
-      <joint_properties damping="1.0" friction="1.0" />
-  </joint>
-  <xacro:wheel position="front" side="right" parent="base" wheel_r="${wheel_r}" wheel_width="${wheel_width}"  base_length="${base_length}" base_width="${base_width}"/>
-  <xacro:wheel position="front" side="left" parent="base" wheel_r="${wheel_r}" wheel_width="${wheel_width}"  base_length="${base_length}" base_width="${base_width}"/>
-  <xacro:wheel position="back" side="right" parent="extension" wheel_r="${wheel_r}" wheel_width="${wheel_width}"  base_length="${base_length}" base_width="${base_width}"/>
-  <xacro:wheel position="back" side="left" parent="extension" wheel_r="${wheel_r}" wheel_width="${wheel_width}"  base_length="${base_length}" base_width="${base_width}"/>
+    <xacro:include filename="$(find hybrid_jumping_robot)/urdf/material.xacro"/>
+    <xacro:include filename="$(find hybrid_jumping_robot)/urdf/plugins.gazebo.xacro"/>
+    <xacro:include filename="$(find hybrid_jumping_robot)/urdf/macro.xacro"/>
+    <xacro:include filename="$(find hybrid_jumping_robot)/urdf/transmission.xacro"/>
+    <xacro:property name="wheel_r" value="0.075"/>
+    <xacro:property name="wheel_width" value="0.03"/>
+    <xacro:property name="wheel_mass" value="0.025"/>
+    <xacro:property name="base_length" value="0.25"/>
+    <xacro:property name="base_width" value="0.15"/>
+    <xacro:property name="base_height" value="0.04"/>
+    <xacro:property name="base_mass" value="0.4"/>
+    <xacro:property name="extension_length" value="0.20"/>
+    <xacro:property name="extension_width" value="0.13"/>
+    <xacro:property name="extension_height" value="0.03"/>
+    <xacro:property name="extension_mass" value="0.4"/>
+    <xacro:property name="motor_base_length" value="0.04"/>
+    <xacro:property name="motor_base_width" value="${base_width}"/>
+    <xacro:property name="motor_base_height" value="${base_height}"/>
+    <xacro:property name="motor_base_mass" value="0.4"/>
+    <link name="base">
+        <visual>
+            <geometry>
+                <box size="${base_length} ${base_width}  ${base_height}"/>
+            </geometry>
+            <material name="blue"/>
+        </visual>
+        <collision>
+            <geometry>
+                <box size="${base_length} ${base_width}  ${base_height}"/>
+            </geometry>
+        </collision>
+        <inertial>
+            <mass value="${base_mass}"/>
+            <inertia ixx="0.21666666666666667" ixy="0" ixz="0" iyy="0.8416666666666667" iyz="0"
+                     izz="1.0416666666666665"/>
+        </inertial>
+    </link>
+    <link name="motor_base">
+        <visual>
+            <geometry>
+                <box size="${motor_base_length} ${motor_base_width}  ${motor_base_height}"/>
+            </geometry>
+            <material name="blue"/>
+        </visual>
+        <collision>
+            <geometry>
+                <box size="${base_length} ${base_width}  ${base_height}"/>
+            </geometry>
+        </collision>
+        <xacro:box_inertial mass="${motor_base_mass}" length="${motor_base_length}" width="${motor_base_width}"
+                            height="${motor_base_height}"/>
+    </link>
+    <joint name="base_motor_base_joint" type="fixed">
+        <axis xyz="1 0 0"/>
+        <parent link="base"/>
+        <child link="motor_base"/>
+        <origin xyz="${motor_base_length*0.5+base_length*0.5} 0 0"/>
+    </joint>
+    <link name="extension">
+        <visual>
+            <geometry>
+                <box size="${extension_length} ${extension_width} ${extension_height}"/>
+            </geometry>
+            <material name="red"/>
+        </visual>
+        <collision>
+            <geometry>
+                <box size="${extension_length} ${extension_width} ${extension_height}"/>
+            </geometry>
+        </collision>
+        <inertial>
+            <mass value="${extension_mass}"/>
+            <inertia ixx="0.17627083333333335" ixy="0" ixz="0" iyy="0.8408541666666667" iyz="0"
+                     izz="1.0020833333333334"/>
+        </inertial>
+    </link>
+    <joint name="extension_base_joint" type="prismatic">
+        <axis xyz="1 0 0"/>
+        <parent link="base"/>
+        <child link="extension"/>
+        <origin xyz="-0.1 0 0"/>
+        <limit lower="-0.9" upper="0" effort="10000" velocity="1000"/>
+        <joint_properties damping="1.0" friction="1.0"/>
+    </joint>
+    <xacro:wheel position="front" side="right" parent="motor_base" wheel_r="${wheel_r}" wheel_width="${wheel_width}"
+                 base_length="${motor_base_length}" base_width="${base_width}" mass="${wheel_mass}"/>
+    <xacro:wheel position="front" side="left" parent="motor_base" wheel_r="${wheel_r}" wheel_width="${wheel_width}"
+                 base_length="${motor_base_length}" base_width="${base_width}" mass="${wheel_mass}"/>
+    <xacro:wheel position="back" side="right" parent="extension" wheel_r="${wheel_r}" wheel_width="${wheel_width}"
+                 base_length="${base_length}" base_width="${base_width}" mass="${wheel_mass}"/>
+    <xacro:wheel position="back" side="left" parent="extension" wheel_r="${wheel_r}" wheel_width="${wheel_width}"
+                 base_length="${base_length}" base_width="${base_width}" mass="${wheel_mass}"/>
 </robot>

File: hybrid_jumping_robot/urdf/macro.xacro (robot description, xacro)
@@ -1,5 +1,5 @@
 <?xml version="1.0"?>
 <robot name="hybrid_robotv0_2" xmlns:xacro="http://ros.org/wiki/xacro">
-    <xacro:macro name="wheel" params="position side parent wheel_r wheel_width base_length base_width">
+    <xacro:macro name="wheel" params="position side parent wheel_r wheel_width base_length base_width mass">
       <link name="${position}_${side}_wheel">
           <visual>
@@ -14,11 +14,8 @@
               </geometry>
           </collision>
-          <inertial>
-              <mass value="1"/>
-              <inertia ixx="0.005658333333333333" ixy="0" ixz="0" iyy="0.005658333333333333" iyz="0" izz="0.01125"/>
-          </inertial>
+          <xacro:cylinder_inertial mass="${mass}" height="${wheel_width}" radii="${wheel_r}"/>
       </link>
       <joint name="${position}_${side}_wheel_joint" type="continuous">
-          <xacro:property name="origin_x" value="${base_length/2-0.05}"/>
+          <xacro:property name="origin_x" value="${0}"/>
           <xacro:if value="${position == 'back'}">
               <xacro:property name="origin_x" value="${-(base_length/2-0.05)}"/>
@@ -43,10 +40,10 @@
             <mass value="${mass}"/>
             <inertia
-                    ixx="${0.083*mass*(${width}+${height})}"
+                    ixx="${0.083*mass*(width+height)}"
                     ixy="0.0"
                     ixz="0.0"
-                    iyy="${0.083*mass*(${length}+${height})}"
+                    iyy="${0.083*mass*(length+height)}"
                     iyz="0.0"
-                    izz="${0.083*mass*(${width}+${length})}" />
+                    izz="${0.083*mass*(width+length)}" />
         </inertial>
     </xacro:macro>
@@ -56,10 +53,10 @@
             <mass value="${mass}"/>
             <inertia
-                    ixx="${0.083*mass*(3*${radii}*${radii}+${height}*${height})}"
+                    ixx="${0.083*mass*(3*radii*radii+height*height)}"
                     ixy="0.0"
                     ixz="0.0"
-                    iyy="${0.083*mass*(3*${radii}*${radii}+${height}*${height})}"
+                    iyy="${0.083*mass*(3*radii*radii+height*height)}"
                     iyz="0.0"
-                    izz="${0.5*mass*(${radii}*${radii}))}" />
+                    izz="${0.5*mass*(radii*radii)}" />
         </inertial>
     </xacro:macro>

File: hybrid_jumping_robot/urdf/plugins.gazebo.xacro (robot description, xacro)
@@ -6,4 +6,7 @@
   <gazebo reference="extension">
     <material>Gazebo/Blue</material>
+  </gazebo>
+  <gazebo reference="motor_base">
+    <material>Gazebo/Green</material>
   </gazebo>
   <gazebo reference="front_left_wheel">

Commit message: Added automagic inertial matrix and mass to ext and base

File: hybrid_jumping_robot/urdf/first_modelV0_2.urdf.xacro (robot description, xacro)
@@ -32,9 +32,6 @@
             </geometry>
         </collision>
-        <inertial>
-            <mass value="${base_mass}"/>
-            <inertia ixx="0.21666666666666667" ixy="0" ixz="0" iyy="0.8416666666666667" iyz="0"
-                     izz="1.0416666666666665"/>
-        </inertial>
+        <xacro:box_inertial mass="${base_mass}" length="${base_length}" width="${base_width}"
+                            height="${base_height}"/>
     </link>
     <link name="motor_base">
@@ -71,9 +68,6 @@
             </geometry>
         </collision>
-        <inertial>
-            <mass value="${extension_mass}"/>
-            <inertia ixx="0.17627083333333335" ixy="0" ixz="0" iyy="0.8408541666666667" iyz="0"
-                     izz="1.0020833333333334"/>
-        </inertial>
+        <xacro:box_inertial mass="${extension_mass}" length="${extension_length}" width="${extension_width}"
+                            height="${extension_height}"/>
     </link>
     <joint name="extension_base_joint" type="prismatic">

Commit message: UPDATE: limits on the extension

File: hybrid_jumping_robot/urdf/first_modelV0_2.urdf.xacro (robot description, xacro)
@@ -76,5 +76,5 @@
         <child link="extension"/>
         <origin xyz="-0.1 0 0"/>
-        <limit lower="-0.9" upper="0" effort="10000" velocity="1000"/>
+        <limit lower="-0.045" upper="0" effort="10000" velocity="1000"/>
         <joint_properties damping="1.0" friction="1.0"/>
     </joint>

Commit message: break works!!!!
Added a couple of functions, to display the velocity
Changed the mass of the front wheels

File: hybrid_jumping_robot/urdf/first_modelV0_2.urdf.xacro (robot description, xacro)
@@ -6,6 +6,6 @@
     <xacro:include filename="$(find hybrid_jumping_robot)/urdf/transmission.xacro"/>
     <xacro:property name="wheel_r" value="0.075"/>
-    <xacro:property name="wheel_width" value="0.03"/>
-    <xacro:property name="wheel_mass" value="0.025"/>
+    <xacro:property name="wheel_width" value="0.05"/>
+    <xacro:property name="wheel_mass" value="1.025"/>
     <xacro:property name="base_length" value="0.25"/>
     <xacro:property name="base_width" value="0.15"/>
@@ -76,6 +76,6 @@
         <child link="extension"/>
         <origin xyz="-0.1 0 0"/>
-        <limit lower="-0.9" upper="0" effort="10000" velocity="1000"/>
-        <joint_properties damping="1.0" friction="1.0"/>
+        <limit lower="-0.9" upper="0.0" effort="10000" velocity="1000"/>
+        <joint_properties damping="100.0" friction="0.0"/>
     </joint>
     <xacro:wheel position="front" side="right" parent="motor_base" wheel_r="${wheel_r}" wheel_width="${wheel_width}"

File: hybrid_jumping_robot/urdf/macro.xacro (robot description, xacro)
@@ -14,5 +14,10 @@
                 </geometry>
             </collision>
-            <xacro:cylinder_inertial mass="${mass}" height="${wheel_width}" radii="${wheel_r}"/>
+            <xacro:if value="${position == 'back'}">
+                <xacro:cylinder_inertial mass="${0.025}" height="${wheel_width}" radii="${wheel_r}"/>
+            </xacro:if>
+            <xacro:if value="${position == 'front'}">
+                <xacro:cylinder_inertial mass="${mass}" height="${wheel_width}" radii="${wheel_r}"/>
+            </xacro:if>
         </link>
         <xacro:if value="${position == 'back'}">
@@ -42,5 +47,5 @@
                 <child link="${position}_${side}_wheel"/>
                 <origin xyz="${origin_x} ${origin_y} 0" rpy="${pi/2} 0 0"/>
-                <limit effort="10000" velocity="1000"/>
+                <limit effort="1000000" velocity="1000"/>
                 <joint_properties damping="0.0" friction="10000.0"/>
             </joint>

File: hybrid_jumping_robot/urdf/plugins.gazebo.xacro (robot description, xacro)
@@ -11,13 +11,21 @@
   </gazebo>
   <gazebo reference="front_left_wheel">
+    <mu1>1.0</mu1>
+    <mu2>1.0</mu2>
     <material>drc/san_fauxcity_sign</material>
   </gazebo>
   <gazebo reference="front_right_wheel">
+    <mu1>1.0</mu1>
+    <mu2>1.0</mu2>
     <material>drc/san_fauxcity_sign</material>
   </gazebo>
   <gazebo reference="back_left_wheel">
+    <mu1>0.2</mu1>
+    <mu2>0.2</mu2>
     <material>drc/san_fauxcity_sign</material>
   </gazebo>
   <gazebo reference="back_right_wheel">
+    <mu1>0.2</mu1>
+    <mu2>0.2</mu2>
     <material>drc/san_fauxcity_sign</material>
   </gazebo>

Commit message: Change mass on front wheels
to 300 g 

Velocity 292.5 cm/minute
 Rpm 30.630528372500482

File: hybrid_jumping_robot/urdf/first_modelV0_2.urdf.xacro (robot description, xacro)
@@ -7,5 +7,5 @@
     <xacro:property name="wheel_r" value="0.075"/>
     <xacro:property name="wheel_width" value="0.05"/>
-    <xacro:property name="wheel_mass" value="1.025"/>
+    <xacro:property name="wheel_mass" value="0.3"/>
     <xacro:property name="base_length" value="0.25"/>
     <xacro:property name="base_width" value="0.15"/>

Commit message: Changed size to new layout
wheel radii is also very important

File: hybrid_jumping_robot/urdf/first_modelV0_2.urdf.xacro (robot description, xacro)
@@ -8,13 +8,13 @@
     <xacro:property name="wheel_width" value="0.05"/>
     <xacro:property name="wheel_mass" value="0.3"/>
-    <xacro:property name="base_length" value="0.25"/>
-    <xacro:property name="base_width" value="0.15"/>
-    <xacro:property name="base_height" value="0.04"/>
+    <xacro:property name="base_length" value="0.215"/>
+    <xacro:property name="base_width" value="0.1772"/>
+    <xacro:property name="base_height" value="0.0801"/>
     <xacro:property name="base_mass" value="0.4"/>
     <xacro:property name="extension_length" value="0.20"/>
-    <xacro:property name="extension_width" value="0.13"/>
-    <xacro:property name="extension_height" value="0.03"/>
+    <xacro:property name="extension_width" value="0.1581"/>
+    <xacro:property name="extension_height" value="0.0601"/>
     <xacro:property name="extension_mass" value="0.4"/>
-    <xacro:property name="motor_base_length" value="0.04"/>
+    <xacro:property name="motor_base_length" value="0.0585"/>
     <xacro:property name="motor_base_width" value="${base_width}"/>
     <xacro:property name="motor_base_height" value="${base_height}"/>

Commit message: UPDATE: fix collision #34

File: hybrid_jumping_robot/urdf/first_modelV0_2.urdf.xacro (robot description, xacro)
@@ -44,5 +44,5 @@
         <collision>
             <geometry>
-                <box size="${base_length} ${base_width}  ${base_height}"/>
+                <box size="${motor_base_length} ${motor_base_width}  ${motor_base_height}"/>
             </geometry>
         </collision>

Commit message: UPDATE: obtain the velocity feedback #89

File: hybrid_jumping_robot/urdf/first_modelV0_2.urdf.xacro (robot description, xacro)
@@ -8,4 +8,5 @@
     <xacro:property name="wheel_width" value="0.05"/>
     <xacro:property name="wheel_mass" value="0.3"/>
+    <xacro:property name="wheel_back_mass" value="0.05"/>
     <xacro:property name="base_length" value="0.215"/>
     <xacro:property name="base_width" value="0.1772"/>
@@ -83,7 +84,7 @@
     <xacro:wheel position="front" side="left" parent="motor_base" wheel_r="${wheel_r}" wheel_width="${wheel_width}"
                  base_length="${motor_base_length}" base_width="${base_width}" mass="${wheel_mass}"/>
+    <xacro:wheel position="back" side="left" parent="extension" wheel_r="${wheel_r}" wheel_width="${wheel_width}"
+                 base_length="${base_length}" base_width="${base_width}" mass="${wheel_back_mass}"/>
     <xacro:wheel position="back" side="right" parent="extension" wheel_r="${wheel_r}" wheel_width="${wheel_width}"
-                 base_length="${base_length}" base_width="${base_width}" mass="${wheel_mass}"/>
-    <xacro:wheel position="back" side="left" parent="extension" wheel_r="${wheel_r}" wheel_width="${wheel_width}"
-                 base_length="${base_length}" base_width="${base_width}" mass="${wheel_mass}"/>
+                 base_length="${base_length}" base_width="${base_width}" mass="${wheel_back_mass}"/>
 </robot>
