Commit message: Added inertial matrixes to macros
easier method of getting the inertial matrix

File: hybrid_jumping_robot/urdf/macro.xacro (robot description, xacro)
@@ -1,5 +1,5 @@
 <?xml version="1.0"?>
 <robot name="hybrid_robotv0_2" xmlns:xacro="http://ros.org/wiki/xacro">
-  <xacro:macro name="wheel" params="position side parent wheel_r wheel_width base_length base_width">
+    <xacro:macro name="wheel" params="position side parent wheel_r wheel_width base_length base_width">
       <link name="${position}_${side}_wheel">
           <visual>
@@ -37,4 +37,30 @@
           <joint_properties damping="1.0" friction="1.0" />
       </joint>
-  </xacro:macro>
+    </xacro:macro>
+    <!--box_inertial makes it easier to implement mass and inertial for a box shape-->
+    <xacro:macro name="box_inertial" params="mass length width height">
+        <inertial>
+            <mass value="${mass}"/>
+            <inertia
+                    ixx="${0.083*mass*(${width}+${height})}"
+                    ixy="0.0"
+                    ixz="0.0"
+                    iyy="${0.083*mass*(${length}+${height})}"
+                    iyz="0.0"
+                    izz="${0.083*mass*(${width}+${length})}" />
+        </inertial>
+    </xacro:macro>
+    <!--cylinder_inertial makes it easier to implement mass and inertial for a cylinder shape-->
+    <xacro:macro name="cylinder_inertial" params="mass height radii">
+        <inertial>
+            <mass value="${mass}"/>
+            <inertia
+                    ixx="${0.083*mass*(3*${radii}*${radii}+${height}*${height})}"
+                    ixy="0.0"
+                    ixz="0.0"
+                    iyy="${0.083*mass*(3*${radii}*${radii}+${height}*${height})}"
+                    iyz="0.0"
+                    izz="${0.5*mass*(${radii}*${radii}))}" />
+        </inertial>
+    </xacro:macro>
 </robot>

Commit message: Changed the friction to zero on the back wheels

File: hybrid_jumping_robot/urdf/macro.xacro (robot description, xacro)
@@ -2,36 +2,47 @@
 <robot name="hybrid_robotv0_2" xmlns:xacro="http://ros.org/wiki/xacro">
     <xacro:macro name="wheel" params="position side parent wheel_r wheel_width base_length base_width mass">
-      <link name="${position}_${side}_wheel">
-          <visual>
-              <geometry>
-                  <cylinder radius="${wheel_r}" length="${wheel_width}"/>
-              </geometry>
-              <material name="black"/>
-          </visual>
-          <collision>
-              <geometry>
-                  <cylinder radius="${wheel_r}" length="${wheel_width}"/>
-              </geometry>
-          </collision>
-          <xacro:cylinder_inertial mass="${mass}" height="${wheel_width}" radii="${wheel_r}"/>
-      </link>
-      <joint name="${position}_${side}_wheel_joint" type="continuous">
-          <xacro:property name="origin_x" value="${0}"/>
-          <xacro:if value="${position == 'back'}">
-              <xacro:property name="origin_x" value="${-(base_length/2-0.05)}"/>
-          </xacro:if>
-          <xacro:property name="origin_y" value="${(base_width + wheel_width)/2}"/>
-          <xacro:if value="${side == 'right'}">
-              <xacro:property name="origin_y" value="${-(base_width + wheel_width)/2}"/>
-          </xacro:if>
-          <xacro:if value="${parent == 'extension'}">
-          </xacro:if>
-          <axis xyz="0 0 1" rpy="0 0 0"/>
-          <parent link="${parent}"/>
-          <child link="${position}_${side}_wheel"/>
-          <origin xyz="${origin_x} ${origin_y} 0" rpy="${pi/2} 0 0"/>
-          <limit effort="10000" velocity="1000"/>
-          <joint_properties damping="1.0" friction="1.0" />
-      </joint>
+        <link name="${position}_${side}_wheel">
+            <visual>
+                <geometry>
+                    <cylinder radius="${wheel_r}" length="${wheel_width}"/>
+                </geometry>
+                <material name="black"/>
+            </visual>
+            <collision>
+                <geometry>
+                    <cylinder radius="${wheel_r}" length="${wheel_width}"/>
+                </geometry>
+            </collision>
+            <xacro:cylinder_inertial mass="${mass}" height="${wheel_width}" radii="${wheel_r}"/>
+        </link>
+        <xacro:if value="${position == 'back'}">
+            <joint name="${position}_${side}_wheel_joint" type="continuous">
+                <xacro:property name="origin_x" value="${-(base_length/2-0.05)}"/>
+                <xacro:property name="origin_y" value="${(base_width + wheel_width)/2}"/>
+                <xacro:if value="${side == 'right'}">
+                    <xacro:property name="origin_y" value="${-(base_width + wheel_width)/2}"/>
+                </xacro:if>
+                <axis xyz="0 0 1" rpy="0 0 0"/>
+                <parent link="${parent}"/>
+                <child link="${position}_${side}_wheel"/>
+                <origin xyz="${origin_x} ${origin_y} 0" rpy="${pi/2} 0 0"/>
+                <joint_properties damping="0.0" friction="0.0"/>
+            </joint>
+        </xacro:if>
+        <xacro:if value="${position == 'front'}">
+            <joint name="${position}_${side}_wheel_joint" type="continuous">
+                <xacro:property name="origin_x" value="${0}"/>
+                <xacro:property name="origin_y" value="${(base_width + wheel_width)/2}"/>
+                <xacro:if value="${side == 'right'}">
+                    <xacro:property name="origin_y" value="${-(base_width + wheel_width)/2}"/>
+                </xacro:if>
+                <axis xyz="0 0 1" rpy="0 0 0"/>
+                <parent link="${parent}"/>
+                <child link="${position}_${side}_wheel"/>
+                <origin xyz="${origin_x} ${origin_y} 0" rpy="${pi/2} 0 0"/>
+                <limit effort="10000" velocity="1000"/>
+                <joint_properties damping="1.0" friction="1.0"/>
+            </joint>
+        </xacro:if>
     </xacro:macro>
     <!--box_inertial makes it easier to implement mass and inertial for a box shape-->
@@ -45,5 +56,5 @@
                     iyy="${1/12*mass*(length*length+height*height)}"
                     iyz="0.0"
-                    izz="${1/12*mass*(width*width+length*length)}" />
+                    izz="${1/12*mass*(width*width+length*length)}"/>
         </inertial>
     </xacro:macro>
@@ -58,5 +69,5 @@
                     iyy="${1/12*mass*(3*radii*radii+height*height)}"
                     iyz="0.0"
-                    izz="${0.5*mass*(radii*radii)}" />
+                    izz="${0.5*mass*(radii*radii)}"/>
         </inertial>
     </xacro:macro>

Commit message: UPDATE: set non-driven wheels to move freely

File: hybrid_jumping_robot/urdf/macro.xacro (robot description, xacro)
@@ -28,4 +28,5 @@
                 <origin xyz="${origin_x} ${origin_y} 0" rpy="${pi/2} 0 0"/>
                 <joint_properties damping="0.0" friction="0.0"/>
+                <limit effort="0.0" velocity="100000.0"/>
             </joint>
         </xacro:if>

Commit message: UPDATE: correct inertia and mass wheels added #95 still missing the rest of inertias update

File: hybrid_jumping_robot/urdf/macro.xacro (robot description, xacro)
@@ -18,10 +18,10 @@
                 <inertial>
                     <mass value="${mass}"/>
-                    <inertia ixx="181652.29"
+                    <inertia ixx="${181652.29/1000000000}"
                              ixy="0.0"
                              ixz="0.0"
-                             iyy="181652.29"
+                             iyy="${181652.29/1000000000}"
                              iyz="0.0"
-                             izz="361145.59"/>
+                             izz="${361145.59/1000000000}"/>
                 </inertial>
             </xacro:if>
@@ -30,10 +30,10 @@
                 <inertial>
                     <mass value="${mass}"/>
-                    <inertia ixx="528551.19"
+                    <inertia ixx="${528551.19/1000000000}"
                              ixy="0.0"
                              ixz="0.0"
-                             iyy="528551.19"
+                             iyy="${528551.19/1000000000}"
                              iyz="0.0"
-                             izz="1050820.37"/>
+                             izz="${1050820.37/1000000000}"/>
                 </inertial>
             </xacro:if>
