Commit message: UPDATE: add motor #95

File: hybrid_jumping_robot/urdf/last_model.urdf.xacro (robot description, xacro)
@@ -61,3 +61,24 @@
     <origin xyz="${-(base_high_length+base_short_length)*0.5} 0 0"/>
   </joint>
+  <link name="motor_base">
+    <visual>
+      <geometry>
+        <box size="${motor_base_length} ${motor_base_width}  ${motor_base_height}"/>
+      </geometry>
+      <material name="blue"/>
+    </visual>
+    <collision>
+      <geometry>
+        <box size="${motor_base_length} ${motor_base_width}  ${motor_base_height}"/>
+      </geometry>
+    </collision>
+    <xacro:box_inertial mass="${motor_base_mass}" length="${motor_base_length}" width="${motor_base_width}"
+                        height="${motor_base_height}"/>
+  </link>
+  <joint name="base_motor_base_joint" type="fixed">
+    <axis xyz="1 0 0"/>
+    <parent link="base_high"/>
+    <child link="motor_base"/>
+    <origin xyz="${motor_base_length*0.5+base_high_length*0.5} 0 0"/>
+  </joint>
 </robot>

File: hybrid_jumping_robot/urdf/plugins_v2.gazebo.xacro (robot description, xacro)
@@ -7,3 +7,6 @@
     <material>Gazebo/Blue</material>
   </gazebo>
+  <gazebo reference="motor_base">
+    <material>Gazebo/Red</material>
+  </gazebo>
 </robot>

Commit message: UPDATE: final pre-model #95 missing measures and mass

File: hybrid_jumping_robot/urdf/last_model.urdf.xacro (robot description, xacro)
@@ -4,5 +4,5 @@
   <xacro:include filename="$(find hybrid_jumping_robot)/urdf/plugins_v2.gazebo.xacro"/>
   <xacro:include filename="$(find hybrid_jumping_robot)/urdf/macro.xacro"/>
-  <xacro:include filename="$(find hybrid_jumping_robot)/urdf/transmission.xacro"/>
+  <xacro:include filename="$(find hybrid_jumping_robot)/urdf/transmission_v2.xacro"/>
   <!-- Wheels -->
   <xacro:property name="wheel_r" value="0.075"/>
@@ -18,5 +18,5 @@
   <!-- Short part -->
   <xacro:property name="base_short_height" value="0.02"/>
-  <xacro:property name="base_short_length" value="0.1"/>
+  <xacro:property name="base_short_length" value="0.15"/>
   <xacro:property name="base_short_mass" value="0.2"/>
   <!-- Motor -->
@@ -82,3 +82,11 @@
     <origin xyz="${motor_base_length*0.5+base_high_length*0.5} 0 0"/>
   </joint>
+  <xacro:wheel position="front" side="right" parent="motor_base" wheel_r="${wheel_r}" wheel_width="${wheel_width}"
+               base_length="${motor_base_length}" base_width="${base_width}" mass="${front_wheel_mass}"/>
+  <xacro:wheel position="front" side="left" parent="motor_base" wheel_r="${wheel_r}" wheel_width="${wheel_width}"
+               base_length="${motor_base_length}" base_width="${base_width}" mass="${front_wheel_mass}"/>
+  <xacro:wheel position="back" side="right" parent="base_short" wheel_r="${wheel_r}" wheel_width="${wheel_width}"
+               base_length="${base_short_length}" base_width="${base_width}" mass="${back_wheel_mass}"/>
+  <xacro:wheel position="back" side="left" parent="base_short" wheel_r="${wheel_r}" wheel_width="${wheel_width}"
+               base_length="${base_short_length}" base_width="${base_width}" mass="${back_wheel_mass}"/>
 </robot>

File: hybrid_jumping_robot/urdf/macro.xacro (robot description, xacro)
@@ -23,5 +23,5 @@
         <xacro:if value="${position == 'back'}">
             <joint name="${position}_${side}_wheel_joint" type="continuous">
-                <xacro:property name="origin_x" value="${-(base_length/2-0.05)}"/>
+                <xacro:property name="origin_x" value="${-(base_length/2-0.005)}"/>
                 <xacro:property name="origin_y" value="${(base_width + wheel_width)/2}"/>
                 <xacro:if value="${side == 'right'}">

File: hybrid_jumping_robot/urdf/plugins_v2.gazebo.xacro (robot description, xacro)
@@ -10,3 +10,48 @@
     <material>Gazebo/Red</material>
   </gazebo>
+  <gazebo reference="front_left_wheel">
+    <mu1>1.0</mu1>
+    <mu2>1.0</mu2>
+    <material>drc/san_fauxcity_sign</material>
+  </gazebo>
+  <gazebo reference="front_right_wheel">
+    <mu1>1.0</mu1>
+    <mu2>1.0</mu2>
+    <material>drc/san_fauxcity_sign</material>
+  </gazebo>
+  <gazebo reference="back_left_wheel">
+    <mu1>0.2</mu1>
+    <mu2>0.2</mu2>
+    <material>drc/san_fauxcity_sign</material>
+  </gazebo>
+  <gazebo reference="back_right_wheel">
+    <mu1>0.2</mu1>
+    <mu2>0.2</mu2>
+    <material>drc/san_fauxcity_sign</material>
+  </gazebo>
+  <gazebo>
+    <plugin filename="libgazebo_ros_control.so" name="gazebo_ros_control">
+      <robotNamespace>/hybrid_robotV0_2</robotNamespace>
+    </plugin>
+  </gazebo>
+  <gazebo reference="base_short">
+    <gravity>true</gravity>
+    <sensor name="imu_sensor" type="imu">
+      <always_on>true</always_on>
+      <update_rate>1000</update_rate>
+      <visualize>true</visualize>
+      <topic>__default_topic__</topic>
+      <plugin filename="libgazebo_ros_imu_sensor.so" name="imu_plugin">
+        <topicName>imu</topicName>
+        <bodyName>imu_link</bodyName>
+        <updateRateHZ>280.0</updateRateHZ>
+        <gaussianNoise>0.0</gaussianNoise>
+        <xyzOffset>0 0 0</xyzOffset>
+        <rpyOffset>0 0 0</rpyOffset>
+        <frameName>imu_link</frameName>
+        <initialOrientationAsReference>false</initialOrientationAsReference>
+      </plugin>
+      <pose>0 0 0 0 0 0</pose>
+    </sensor>
+  </gazebo>
 </robot>

Commit message: UPDATE: model with correct dimensions #95 The body with the correct dimensions Wheels with the correct width Some clearance between the wheels and the car

File: hybrid_jumping_robot/urdf/last_model.urdf.xacro (robot description, xacro)
@@ -7,5 +7,5 @@
   <!-- Wheels -->
   <xacro:property name="wheel_r" value="0.075"/>
-  <xacro:property name="wheel_width" value="0.05"/>
+  <xacro:property name="wheel_width" value="0.015"/>
   <xacro:property name="front_wheel_mass" value="0.3"/>
   <xacro:property name="back_wheel_mass" value="0.3"/>
@@ -14,9 +14,9 @@
   <!-- High part -->
   <xacro:property name="base_high_height" value="0.0801"/>
-  <xacro:property name="base_high_length" value="0.02"/>
+  <xacro:property name="base_high_length" value="0.01"/>
   <xacro:property name="base_high_mass" value="0.2"/>
   <!-- Short part -->
-  <xacro:property name="base_short_height" value="0.02"/>
-  <xacro:property name="base_short_length" value="0.15"/>
+  <xacro:property name="base_short_height" value="0.012"/>
+  <xacro:property name="base_short_length" value="0.14"/>
   <xacro:property name="base_short_mass" value="0.2"/>
   <!-- Motor -->

File: hybrid_jumping_robot/urdf/macro.xacro (robot description, xacro)
@@ -21,10 +21,11 @@
             </xacro:if>
         </link>
+        <xacro:property name="clear" value="0.009"/>
         <xacro:if value="${position == 'back'}">
             <joint name="${position}_${side}_wheel_joint" type="continuous">
-                <xacro:property name="origin_x" value="${-(base_length/2-0.005)}"/>
-                <xacro:property name="origin_y" value="${(base_width + wheel_width)/2}"/>
+                <xacro:property name="origin_x" value="${-(base_length/2-0.010)}"/>
+                <xacro:property name="origin_y" value="${(base_width + wheel_width)/2 + clear}"/>
                 <xacro:if value="${side == 'right'}">
-                    <xacro:property name="origin_y" value="${-(base_width + wheel_width)/2}"/>
+                    <xacro:property name="origin_y" value="${-(base_width + wheel_width)/2 - clear}"/>
                 </xacro:if>
                 <axis xyz="0 0 1" rpy="0 0 0"/>
@@ -39,7 +40,7 @@
             <joint name="${position}_${side}_wheel_joint" type="continuous">
                 <xacro:property name="origin_x" value="${0}"/>
-                <xacro:property name="origin_y" value="${(base_width + wheel_width)/2}"/>
+                <xacro:property name="origin_y" value="${(base_width + wheel_width)/2 + clear}"/>
                 <xacro:if value="${side == 'right'}">
-                    <xacro:property name="origin_y" value="${-(base_width + wheel_width)/2}"/>
+                    <xacro:property name="origin_y" value="${-(base_width + wheel_width)/2 - clear}"/>
                 </xacro:if>
                 <axis xyz="0 0 1" rpy="0 0 0"/>

Commit message: UPDATE: inertia and mass wheels added #95 still missing the rest of inertias update

File: hybrid_jumping_robot/urdf/last_model.urdf.xacro (robot description, xacro)
@@ -8,6 +8,6 @@
   <xacro:property name="wheel_r" value="0.075"/>
   <xacro:property name="wheel_width" value="0.015"/>
-  <xacro:property name="front_wheel_mass" value="0.3"/>
-  <xacro:property name="back_wheel_mass" value="0.3"/>
+  <xacro:property name="front_wheel_mass" value="0.279"/>
+  <xacro:property name="back_wheel_mass" value="0.09589"/>
   <!-- Body -->
   <xacro:property name="base_width" value="0.1772"/>

File: hybrid_jumping_robot/urdf/macro.xacro (robot description, xacro)
@@ -15,8 +15,26 @@
             </collision>
             <xacro:if value="${position == 'back'}">
-                <xacro:cylinder_inertial mass="${0.025}" height="${wheel_width}" radii="${wheel_r}"/>
+<!--                <xacro:cylinder_inertial mass="${0.025}" height="${wheel_width}" radii="${wheel_r}"/>-->
+                <inertial>
+                    <mass value="${mass}"/>
+                    <inertia ixx="181652.29"
+                             ixy="0.0"
+                             ixz="0.0"
+                             iyy="181652.29"
+                             iyz="0.0"
+                             izz="361145.59"/>
+                </inertial>
             </xacro:if>
             <xacro:if value="${position == 'front'}">
-                <xacro:cylinder_inertial mass="${mass}" height="${wheel_width}" radii="${wheel_r}"/>
+<!--                <xacro:cylinder_inertial mass="${mass}" height="${wheel_width}" radii="${wheel_r}"/>-->
+                <inertial>
+                    <mass value="${mass}"/>
+                    <inertia ixx="528551.19"
+                             ixy="0.0"
+                             ixz="0.0"
+                             iyy="528551.19"
+                             iyz="0.0"
+                             izz="1050820.37"/>
+                </inertial>
             </xacro:if>
         </link>

Commit message: UPDATE: all the inertial done #95 maybe the inertias on the motor have to be moved around (axis change)

File: hybrid_jumping_robot/urdf/last_model.urdf.xacro (robot description, xacro)
@@ -15,14 +15,14 @@
   <xacro:property name="base_high_height" value="0.0801"/>
   <xacro:property name="base_high_length" value="0.01"/>
-  <xacro:property name="base_high_mass" value="0.2"/>
+  <xacro:property name="base_high_mass" value="0.017062817412333738"/>
   <!-- Short part -->
   <xacro:property name="base_short_height" value="0.012"/>
   <xacro:property name="base_short_length" value="0.14"/>
-  <xacro:property name="base_short_mass" value="0.2"/>
+  <xacro:property name="base_short_mass" value="0.035787182587666264"/>
   <!-- Motor -->
   <xacro:property name="motor_base_length" value="0.0585"/>
   <xacro:property name="motor_base_width" value="${base_width}"/>
   <xacro:property name="motor_base_height" value="${base_high_height}"/>
-  <xacro:property name="motor_base_mass" value="0.4"/>
+  <xacro:property name="motor_base_mass" value="0.73466"/>
   <link name="base_high">
     <visual>
@@ -73,6 +73,15 @@
       </geometry>
     </collision>
-    <xacro:box_inertial mass="${motor_base_mass}" length="${motor_base_length}" width="${motor_base_width}"
-                        height="${motor_base_height}"/>
+<!--    <xacro:box_inertial mass="${motor_base_mass}" length="${motor_base_length}" width="${motor_base_width}"-->
+<!--                        height="${motor_base_height}"/>-->
+    <inertial>
+      <mass value="${motor_base_mass}"/>
+      <inertia ixx="${178281296.78/1000000000}"
+               ixy="${17082829.61/1000000000}"
+               ixz="${15751727.91/1000000000}"
+               iyy="${87803241.16/1000000000}"
+               iyz="${88582169.30/1000000000}"
+               izz="${102100565.99/1000000000}"/>
+    </inertial>
   </link>
   <joint name="base_motor_base_joint" type="fixed">

Commit message: UPDATE: motor inertia #95

File: hybrid_jumping_robot/urdf/last_model.urdf.xacro (robot description, xacro)
@@ -77,10 +77,16 @@
     <inertial>
       <mass value="${motor_base_mass}"/>
-      <inertia ixx="${178281296.78/1000000000}"
-               ixy="${17082829.61/1000000000}"
-               ixz="${15751727.91/1000000000}"
-               iyy="${87803241.16/1000000000}"
-               iyz="${88582169.30/1000000000}"
-               izz="${102100565.99/1000000000}"/>
+<!--      <inertia ixx="${178281296.78/1000000000}"-->
+<!--               ixy="${17082829.61/1000000000}"-->
+<!--               ixz="${15751727.91/1000000000}"-->
+<!--               iyy="${87803241.16/1000000000}"-->
+<!--               iyz="${88582169.30/1000000000}"-->
+<!--               izz="${102100565.99/1000000000}"/>-->
+      <inertia ixx="0.00308579"
+               ixy="0.0"
+               ixz="0.0"
+               iyy="0.00059331"
+               iyz="0.0"
+               izz="0.00305473"/>
     </inertial>
   </link>
